Commit message: Fix references to RASberry

File: bacchus_gazebo/urdf/materials/materials.xacro (robot description, xacro)
@@ -1,29 +1,29 @@
 <?xml version="1.0"?>
 <robot>
-  <material name="rasberry/black">
+  <material name="bacchus/black">
     <color rgba="0.0 0.0 0.0 1.0"/>
   </material>
-  <material name="rasberry/blue">
+  <material name="bacchus/blue">
     <color rgba="0.0 0.0 0.8 1.0"/>
   </material>
-  <material name="rasberry/green">
+  <material name="bacchus/green">
     <color rgba="0.0 0.8 0.0 1.0"/>
   </material>
-  <material name="rasberry/grey">
+  <material name="bacchus/grey">
     <color rgba="0.2 0.2 0.2 1.0"/>
   </material>
-  <material name="rasberry/orange">
+  <material name="bacchus/orange">
     <color rgba="${255/255} ${108/255} ${10/255} 1.0"/>
   </material>
-  <material name="rasberry/brown">
+  <material name="bacchus/brown">
     <color rgba="${222/255} ${207/255} ${195/255} 1.0"/>
   </material>
-  <material name="rasberry/red">
+  <material name="bacchus/red">
     <color rgba="0.8 0.0 0.0 1.0"/>
   </material>
-  <material name="rasberry/white">
+  <material name="bacchus/white">
     <color rgba="1.0 1.0 1.0 1.0"/>
   </material>
-  <material name="rasberry/alu">
+  <material name="bacchus/alu">
     <color rgba="0.75 0.75 0.75 1.0"/>
   </material>

File: bacchus_gazebo/urdf/saga_sensors.xacro (robot description, xacro)
@@ -61,5 +61,5 @@
         <xacro:if value="${current_camera in base_params['cameras']}" >
             <xacro:property name="params" value="${base_params['cameras'][current_camera]}" />
-            <xacro:include filename="$(find rasberry_bringup)/urdf/components/sensors/camera_${params['type']}_${params['make']}_${params['model']}/camera_${params['type']}_${params['make']}_${params['model']}.xacro" />
+            <xacro:include filename="$(find bacchus_gazebo)/urdf/sensors/camera_${params['type']}_${params['make']}_${params['model']}/camera_${params['type']}_${params['make']}_${params['model']}.xacro" />
             <xacro:property name="next_camera" value="camera${current_index + 1}" />
             <xacro:if value="${next_camera in base_params['cameras']}" >

File: bacchus_gazebo/urdf/sensors/camera_3d_zed_zed2/camera_3d_zed_zed2.xacro (robot description, xacro)
@@ -17,5 +17,5 @@
 <robot name="camera_3d_zed_zed2_sensor" xmlns:xacro="http://ros.org/wiki/xacro">
     <!--File includes-->
-    <xacro:include filename="$(find rasberry_bringup)/urdf/components/sensors/camera_3d_zed_zed2/zed_zed2.gazebo.xacro"/>
+    <xacro:include filename="$(find bacchus_gazebo)/urdf/sensors/camera_3d_zed_zed2/zed_zed2.gazebo.xacro"/>
     <!-- Properties -->
     <xacro:property name="M_PI"     value="3.1415926535897931" />

File: bacchus_gazebo/urdf/sensors/gnss_antenna_generic/gnss_antenna.macro.xacro (robot description, xacro)
@@ -1,5 +1,5 @@
 <?xml version="1.0"?>
 <robot xmlns:xacro="http://www.ros.org/wiki/xacro">
-  <xacro:include filename="$(find rasberry_bringup)/urdf/components/sensors/gnss_antenna_generic/gnss_antenna.gazebo.xacro"/>
+  <xacro:include filename="$(find bacchus_gazebo)/urdf/sensors/gnss_antenna_generic/gnss_antenna.gazebo.xacro"/>
   <xacro:macro name="gnss_antenna_sensor" params="tf_prefix parent_link output_sim suffix datum_file *joint_pose">
     <link name="${tf_prefix}gps_${suffix}" >

File: bacchus_gazebo/urdf/sensors/gnss_antenna_generic/gnss_antenna.xacro (robot description, xacro)
@@ -1,5 +1,5 @@
 <?xml version="1.0"?>
 <robot xmlns:xacro="http://www.ros.org/wiki/xacro">
-  <xacro:include filename="$(find rasberry_bringup)/urdf/components/sensors/gnss_antenna_generic/gnss_antenna.gazebo.xacro"/>
+  <xacro:include filename="$(find bacchus_gazebo)/urdf/sensors/gnss_antenna_generic/gnss_antenna.gazebo.xacro"/>
     <link name="${tf_prefix}gps_${params['suffix']}" >
       <visual>

File: bacchus_gazebo/urdf/sensors/imu_um7/imu_um7.macro.xacro (robot description, xacro)
@@ -1,5 +1,5 @@
 <?xml version="1.0"?>
 <robot xmlns:xacro="http://www.ros.org/wiki/xacro">
-  <xacro:include filename="$(find rasberry_bringup)/urdf/components/sensors/imu_um7/imu_um7.gazebo.xacro"/>
+  <xacro:include filename="$(find bacchus_gazebo)/urdf/sensors/imu_um7/imu_um7.gazebo.xacro"/>
   <xacro:macro name="imu_um7_sensor" params="tf_prefix parent_link *joint_pose">
     <link name="${tf_prefix}imu_link"/>

File: bacchus_gazebo/urdf/sensors/imu_um7/imu_um7.xacro (robot description, xacro)
@@ -1,5 +1,5 @@
 <?xml version="1.0"?>
 <robot xmlns:xacro="http://www.ros.org/wiki/xacro">
-    <xacro:include filename="$(find rasberry_bringup)/urdf/components/sensors/imu_um7/imu_um7.gazebo.xacro"/>
+    <xacro:include filename="$(find bacchus_gazebo)/urdf/sensors/imu_um7/imu_um7.gazebo.xacro"/>
     <link name="${tf_prefix}imu_link"/>
     <joint name="base_sens_imu" type="fixed">

File: bacchus_gazebo/urdf/sensors/laserscanner_3d_ouster_os1/laserscanner_3d_ouster_os1.xacro (robot description, xacro)
@@ -1,5 +1,5 @@
 <?xml version="1.0"?>
 <robot xmlns:xacro="http://www.ros.org/wiki/xacro">
-  <xacro:include filename="$(find rasberry_bringup)/urdf/components/sensors/laserscanner_3d_ouster_os1/laserscanner_3d_ouster_os1.gazebo.xacro"/>
+  <xacro:include filename="$(find bacchus_gazebo)/urdf/sensors/laserscanner_3d_ouster_os1/laserscanner_3d_ouster_os1.gazebo.xacro"/>
     <link name="${tf_prefix}os1_${params['suffix']}">
       <collision>

File: bacchus_gazebo/urdf/sensors/laserscanner_3d_sick_mrs1000/laserscanner_3d_sick_mrs1000.macro.xacro (robot description, xacro)
@@ -1,5 +1,5 @@
 <?xml version="1.0"?>
 <robot xmlns:xacro="http://www.ros.org/wiki/xacro">
-  <xacro:include filename="$(find rasberry_bringup)/urdf/components/sensors/laserscanner_3d_sick_mrs1000/laserscanner_3d_sick_mrs1000.gazebo.xacro"/>
+  <xacro:include filename="$(find bacchus_gazebo)/urdf/sensors/laserscanner_3d_sick_mrs1000/laserscanner_3d_sick_mrs1000.gazebo.xacro"/>
   <xacro:macro name="laserscanner_3d_sick_mrs1000_sensor" params="robot_name tf_prefix parent_link output_sim topic_prefix suffix *joint_pose">
     <link name="${tf_prefix}mrs1000_${suffix}_POS_000_DIST1">

File: bacchus_gazebo/urdf/sensors/laserscanner_3d_sick_mrs1000/laserscanner_3d_sick_mrs1000.xacro (robot description, xacro)
@@ -1,5 +1,5 @@
 <?xml version="1.0"?>
 <robot xmlns:xacro="http://www.ros.org/wiki/xacro">
-  <xacro:include filename="$(find rasberry_bringup)/urdf/components/sensors/laserscanner_3d_sick_mrs1000/laserscanner_3d_sick_mrs1000.gazebo.xacro"/>
+  <xacro:include filename="$(find bacchus_gazebo)/urdf/sensors/laserscanner_3d_sick_mrs1000/laserscanner_3d_sick_mrs1000.gazebo.xacro"/>
     <link name="${tf_prefix}mrs1000_${params['suffix']}_POS_000_DIST1">
       <collision>
