Commit message: Update URDF and add sensors

File: bacchus_gazebo/urdf/sensors/camera_3d_zed_s185/camera_3d_zed_s185.xacro (robot description, xacro)
@@ -15,7 +15,7 @@
 OF THIS SOFTWARE, EVEN IF ADVISED OF THE POSSIBILITY OF SUCH DAMAGE.
 -->
-<robot name="camera_3d_zed_zed2_sensor" xmlns:xacro="http://ros.org/wiki/xacro">
+<robot name="camera_3d_zed_s185_sensor" xmlns:xacro="http://ros.org/wiki/xacro">
     <!--File includes-->
-    <xacro:include filename="$(find bacchus_gazebo)/urdf/sensors/camera_3d_zed_zed2/zed_zed2.gazebo.xacro"/>
+    <xacro:include filename="$(find bacchus_gazebo)/urdf/sensors/camera_3d_zed_s185/zed_s185.gazebo.xacro"/>
     <!-- Properties -->
     <xacro:property name="M_PI"     value="3.1415926535897931" />
@@ -31,5 +31,5 @@
             <origin xyz="0 0 0" rpy="0 0 0"/>
             <geometry>
-                <mesh filename="package://bacchus_gazebo/urdf/sensors/camera_3d_zed_zed2/meshes/zed2.stl" />
+                <mesh filename="package://bacchus_gazebo/urdf/sensors/camera_3d_zed_s185/meshes/zed2.stl" />
             </geometry>
         </visual>
@@ -87,5 +87,5 @@
     <link name="${tf_prefix}${params['suffix']}_zed2_temp_right_link" />
     <!-- Camera Gazebo Plugin -->
-    <xacro:camera_3d_zed_zed2_gazebo
+    <xacro:camera_3d_zed_s185_gazebo
         robot_name="${robot_name}"
         tf_prefix="${tf_prefix}"
@@ -93,4 +93,4 @@
         topic_prefix="${params['topic_prefix']}"
         suffix="${params['suffix']}">
-    </xacro:camera_3d_zed_zed2_gazebo>
+    </xacro:camera_3d_zed_s185_gazebo>
 </robot>

File: bacchus_gazebo/urdf/sensors/camera_3d_zed_s185/zed_s185.gazebo.xacro (robot description, xacro)
@@ -6,5 +6,5 @@
 -->
 <robot xmlns:xacro="http://ros.org/wiki/xacro">
-  <xacro:macro name="camera_3d_zed_zed2_gazebo" params="robot_name tf_prefix output_sim topic_prefix suffix" >
+  <xacro:macro name="camera_3d_zed_s185_gazebo" params="robot_name tf_prefix output_sim topic_prefix suffix" >
     <xacro:if value="${output_sim}">
       <!-- Load parameters to model's main link-->
@@ -13,8 +13,8 @@
         <sensor name="${tf_prefix}${suffix}_left_camera_optical_frame" type="camera">
           <camera name="${robot_name}zed2_camera">
-            <horizontal_fov>${88*deg_to_rad}</horizontal_fov>
+            <horizontal_fov>${30*deg_to_rad}</horizontal_fov>
             <image>
-              <width>1920</width>
-              <height>1080</height>
+              <width>1000</width>
+              <height>1000</height>
               <format>RGB_INT8</format>
             </image>
@@ -31,5 +31,5 @@
           <always_on>1</always_on>
           <update_rate>30</update_rate>
-          <visualize>0</visualize>
+          <visualize>1</visualize>
           <plugin name="${topic_prefix}" filename="libgazebo_ros_camera.so">
             <cameraName>${tf_prefix}${suffix}_zed2_camera/left</cameraName>
@@ -41,8 +41,8 @@
         <sensor name="${tf_prefix}${suffix}_right_camera_optical_frame" type="camera">
           <camera name="${robot_name}zed2_camera">
-            <horizontal_fov>${88*deg_to_rad}</horizontal_fov>
+            <horizontal_fov>${30*deg_to_rad}</horizontal_fov>
             <image>
-              <width>1920</width>
-              <height>1080</height>
+              <width>1000</width>
+              <height>1000</height>
               <format>RGB_INT8</format>
             </image>
@@ -59,5 +59,5 @@
           <always_on>1</always_on>
           <update_rate>30</update_rate>
-          <visualize>0</visualize>
+          <visualize>1</visualize>
           <plugin name="${topic_prefix}" filename="libgazebo_ros_camera.so">
             <cameraName>${tf_prefix}${suffix}_zed2/right</cameraName>
@@ -67,7 +67,7 @@
           </plugin>
         </sensor>
-        <sensor name="${tf_prefix}${suffix}_left_camera_optical_frame" type="depth">
+        <!-- <sensor name="${tf_prefix}${suffix}_left_camera_optical_frame" type="depth">
           <camera name="${robot_name}zed2_camera">
-            <horizontal_fov>${69.4*deg_to_rad}</horizontal_fov>
+            <horizontal_fov>${30*deg_to_rad}</horizontal_fov>
             <image>
               <width>1920</width>
@@ -96,5 +96,5 @@
         <sensor name="${tf_prefix}${suffix}_zed2_camera_center" type="depth">
           <camera name="${robot_name}zed2_camera">
-            <horizontal_fov>${85.2*deg_to_rad}</horizontal_fov>
+            <horizontal_fov>${30*deg_to_rad}</horizontal_fov>
             <image>
               <width>1280</width>
@@ -120,5 +120,5 @@
             <frameName>${tf_prefix}${suffix}_zed2_camera_center</frameName>
           </plugin>
-        </sensor>
+        </sensor> -->
       </gazebo>
     </xacro:if>

File: bacchus_gazebo/urdf/sensors/laserscanner_3d_ouster_os1/laserscanner_3d_ouster_os1.xacro (robot description, xacro)
@@ -13,5 +13,5 @@
         <geometry>
           <!-- Use sick stl for now, only affects visualisation -->
-          <mesh filename="package://rasberry_bringup/urdf/components/sensors/laserscanner_3d_sick_mrs1000/meshes/mrs1000.stl"/>
+          <mesh filename="package://bacchus_gazebo/urdf/sensors/laserscanner_3d_sick_mrs1000/meshes/mrs1000.stl"/>
         </geometry>
       </visual>

File: bacchus_gazebo/urdf/sensors/laserscanner_3d_sick_mrs1000/laserscanner_3d_sick_mrs1000.macro.xacro (robot description, xacro)
@@ -13,5 +13,5 @@
         <origin xyz="0 0 0" rpy="0 0 0"/>
         <geometry>
-          <mesh filename="package://rasberry_bringup/urdf/components/sensors/laserscanner_3d_sick_mrs1000/meshes/mrs1000.stl"/>
+          <mesh filename="package://bacchus_gazebo/urdf/sensors/laserscanner_3d_sick_mrs1000/meshes/mrs1000.stl"/>
         </geometry>
       </visual>
@@ -32,5 +32,5 @@
         <origin xyz="0 0 0" rpy="0 0 0"/>
         <geometry>
-          <mesh filename="package://rasberry_bringup/urdf/components/sensors/laserscanner_3d_sick_mrs1000/meshes/mrs1000.stl"/>
+          <mesh filename="package://bacchus_gazebo/urdf/sensors/laserscanner_3d_sick_mrs1000/meshes/mrs1000.stl"/>
         </geometry>
       </visual>

File: bacchus_gazebo/urdf/sensors/laserscanner_3d_sick_mrs1000/laserscanner_3d_sick_mrs1000.xacro (robot description, xacro)
@@ -12,5 +12,5 @@
         <origin xyz="0 0 0" rpy="0 0 0"/>
         <geometry>
-          <mesh filename="package://rasberry_bringup/urdf/components/sensors/laserscanner_3d_sick_mrs1000/meshes/mrs1000.stl"/>
+          <mesh filename="package://bacchus_gazebo/urdf/sensors/laserscanner_3d_sick_mrs1000/meshes/mrs1000.stl"/>
         </geometry>
       </visual>
